Commit message: Completed Day 39 Full Gazebo within 95 hrs

File: src/my_robot_description/urdf/base.xacro (robot description, xacro)
@@ -5,5 +5,5 @@
             <!-- Visual Representation -->
             <visual>
-                <origin xyz="0 0 0.05"/>
+                <origin xyz="0 0 0.15"/>
                 <geometry>
                     <box size="${robot_length} ${robot_width} 0.10"/>

File: src/my_robot_description/urdf/gazebo.xacro (robot description, xacro)
@@ -26,3 +26,32 @@
         </plugin>
     </gazebo>
+    <gazebo reference="lidar_link">
+        <sensor name="lidar_sensor" type="gpu_lidar">
+            <topic>scan</topic>
+            <update_rate>10</update_rate>
+            <always_on>true</always_on>
+            <visualize>true</visualize>
+            <ray>
+            <scan>
+                <horizontal>
+                <samples>360</samples>
+                <resolution>1</resolution>
+                <min_angle>-3.14159</min_angle>
+                <max_angle>3.14159</max_angle>
+                </horizontal>
+                <vertical>
+                <samples>1</samples>
+                <resolution>0.01</resolution>
+                <min_angle>0</min_angle>
+                <max_angle>0</max_angle>
+                </vertical>
+            </scan>
+            <range>
+                <min>0.10</min>
+                <max>10.0</max>
+                <resolution>0.01</resolution>
+            </range>
+            </ray>
+        </sensor>
+        </gazebo>
 </robot>

File: src/my_robot_description/urdf/robot.urdf.xacro (robot description, xacro)
@@ -38,3 +38,4 @@
     <!-- Camera -->
     <xacro:camera/>
+    <xacro:lidar/>
 </robot>

File: src/my_robot_description/urdf/sensors.xacro (robot description, xacro)
@@ -9,13 +9,54 @@
                 <material name="red"/>
             </visual>
+            <collision>
+                <geometry>
+                    <box size="0.05 0.05 0.05"/>
+                </geometry>
+            </collision>
+            <inertial>
+                <mass value="0.05"/>
+                <inertia
+                    ixx="0.00002"
+                    ixy="0.0"
+                    ixz="0.0"
+                    iyy="0.00002"
+                    iyz="0.0"
+                    izz="0.00002"/>
+            </inertial>
         </link>
-        <joint
-            name="camera_joint"
-            type="fixed">
+        <joint name="camera_joint" type="fixed">
             <parent link="base_link"/>
             <child link="camera_link"/>
-            <origin
-                xyz="0.20 0 0.15"
-                rpy="0 0 0"/>
+            <origin xyz="0.20 0 0.15" rpy="0 0 0"/>
+        </joint>
+    </xacro:macro>
+    <xacro:macro name="lidar">
+        <link name="lidar_link">
+            <visual>
+                <geometry>
+                    <cylinder length="0.04" radius="0.03"/>
+                </geometry>
+                <material name="blue"/>
+            </visual>
+            <collision>
+                <geometry>
+                    <cylinder length="0.04" radius="0.03"/>
+                </geometry>
+            </collision>
+            <inertial>
+                <mass value="0.05"/>
+                <inertia
+                    ixx="0.00002"
+                    ixy="0.0"
+                    ixz="0.0"
+                    iyy="0.00002"
+                    iyz="0.0"
+                    izz="0.00002"/>
+            </inertial>
+        </link>
+        <joint name="lidar_joint" type="fixed">
+            <parent link="base_link"/>
+            <child link="lidar_link"/>
+            <origin xyz="0.1 0 0.2" rpy="0 0 0"/>
         </joint>
     </xacro:macro>

File: src/my_robot_description/urdf/wheels.xacro (robot description, xacro)
@@ -47,4 +47,5 @@
             <parent link="${parent}"/>
             <child link="${name}"/>
+            <axis xyz="0 1 0"/>
             <origin
                 xyz="${x} ${y} ${wheel_radius}"
